File: Electronics/2024/TivaWareSeeker/CIRCUITV05.brd (EAGLE design)
At the start: 273 x 160.3 mm, 82 parts, among them IC1 7805TV, Q1 BC548, Q10 IRF520, Q11 BC548, Q12 IRF520, Q2 IRF520, Q3 BC548, Q4 IRF520, Q5 BC548, Q6 IRF520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

Commit message: BoardMiddle
Parts:
- moved D9 93.0 mm to (91.7, -5.41)
- moved LED6 93.0 mm to (101.4, -24.6)
- moved R13 93.0 mm to (93.0, -22.6)
- moved R14 93.0 mm to (92.7, -26.6)
- moved Q11 92.1 mm to (91.6, -16.3), turned to 180 degrees
- moved X3 89.2 mm to (8.97, -49.8)
- moved D4 87.0 mm to (7.08, -4.76)
- moved LED1 87.0 mm to (17.8, -24.6)
- moved Q1 87.0 mm to (6.57, -15.9)
- moved R3 87.0 mm to (8.97, -21.9)
- moved R4 87.0 mm to (8.97, -27.0)
- moved Q2 85.1 mm to (8.97, -33.4)
- moved MOTOR3 78.7 mm to (-59.7, -48.1), flipped to the top, turned to 180 degrees
- moved MOTOR2 71.5 mm to (-78.7, -47.8), turned to 180 degrees
- moved Q12 70.1 mm to (90.4, -33.4)
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Connections:
- new net PMW1: U$1.P20
- net 3V3MOT: no longer MOTORIGHT.2
- net ENDER: now also U$1.P33; no longer U$1.P34
- net ENIZQ: now also U$1.P34; no longer U$1.P33
- net GND@1: now also 5V5AOUT1.10, 5V5AOUT1.12, 5V5AOUT1.14, 5V5AOUT1.16, 5V5AOUT1.18, 5V5AOUT1.2, 5V5AOUT1.20, 5V5AOUT1.4, 5V5AOUT1.6, 5V5AOUT1.8
- net GND@3: no longer MOTORIGHT.1
- net GND@4: no longer 5V5AOUT1.10, 5V5AOUT1.12, 5V5AOUT1.14, 5V5AOUT1.16, 5V5AOUT1.18, 5V5AOUT1.2, 5V5AOUT1.20, 5V5AOUT1.4, 5V5AOUT1.6, 5V5AOUT1.8
- net INA2: now also U$1.P37; no longer U$1.P32
- net INA3: now also U$1.P32; no longer U$1.P37
- net INB2: now also U$1.P36; no longer U$1.P31
- net INB3: now also U$1.P31; no longer U$1.P36
- net PWM1: no longer U$1.P20
Routing:
- net GND@3: track 609.5 -> 22.3 mm
- net 3V3MOT: track 1079.3 -> 656.6 mm
- net PWM1: track 301.8 -> 0.00 mm
- net PWM3: track 295.6 -> 0.00 mm
- net PWM4: track 289.1 -> 0.00 mm
- net GND@1: track 1056.6 -> 905.7 mm, vias 2 -> 0
- net 5V1A: track 234.2 -> 98.7 mm
- net M2: track 132.5 -> 0.00 mm
- net INA2: track 109.3 -> 0.00 mm, vias 2 -> 0
- net INB2: track 109.1 -> 0.00 mm, vias 2 -> 0
- net PWM7: track 92.2 -> 0.00 mm, vias 2 -> 0
- net M1: track 154.6 -> 234.9 mm
- net PWM2: track 301.2 -> 225.3 mm
- net M6: track 73.6 -> 135.3 mm
- net ENIZQ: track 59.3 -> 2.63 mm
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Other:
- board size 273 x 160.3 mm -> 270 x 150.3 mm
