File: Electronics/2024/TivaWareSeeker/CIRCUITV05.sch (EAGLE design)
At the start: 82 parts, among them IC1 7805TV, Q1 BC548, Q10 IRF520, Q11 BC548, Q12 IRF520, Q2 IRF520, Q3 BC548, Q4 IRF520, Q5 BC548, Q6 IRF520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

Commit message: BoardMiddle
Connections:
- net ENDER: now also U$1.PH1; no longer U$1.PH0
- net ENIZQ: now also U$1.PH0; no longer U$1.PH1
- net GND@1: now also 5V5AOUT1.10, 5V5AOUT1.12, 5V5AOUT1.14, 5V5AOUT1.16, 5V5AOUT1.18, 5V5AOUT1.2, 5V5AOUT1.20, 5V5AOUT1.4, 5V5AOUT1.6, 5V5AOUT1.8
- net GND@3: no longer MOTORIGHT.1
- net GND@4: no longer 5V5AOUT1.10, 5V5AOUT1.12, 5V5AOUT1.14, 5V5AOUT1.16, 5V5AOUT1.18, 5V5AOUT1.2, 5V5AOUT1.20, 5V5AOUT1.4, 5V5AOUT1.6, 5V5AOUT1.8
- net INA2: now also U$1.PM0; no longer U$1.PK6
- net INA3: now also U$1.PK6; no longer U$1.PM0
- net INB2: now also U$1.PM1; no longer U$1.PK7
- net INB3: now also U$1.PK7; no longer U$1.PM1
