File: Electronics/2024/TivaWareSeeker/CIRCUIT.brd (EAGLE design)
At the start: 213.3 x 115.2 mm, 29 parts, among them IC1 7805TV, X1 KUSBVX, X3 KUSBVX

Commit message: BoardMiddle
Parts:
- removed JP2, JP3, JP4: (no value), pinhead:2X10
- removed SV1, SV2: (no value), con-lstb:MA10-1
- added 5V5AOUT1: (no value), pinhead:2X10
- added ANALOGS: (no value), con-amp-quick:08PA
- added C8, C9: 0.1uF, rcl:C075-052X106
- added D4, D5, D6, D7, D8, D9: 1N4004, diode:DO41-10
- added F1: 6A, fuse:SHK20L
- added LED1, LED2, LED3, LED4, LED5, LED6: TLLG4400, led:LED3MM
- added MOTOR1, MOTOR2, MOTOR3: (no value), con-amp-quick:07PA
- added MOTORIGHT, MOTORLEFT: (no value), pinhead:2X04
- added Q1, Q11, Q3, Q5, Q7, Q9: BC548, transistor-npn:TO92-EBC
- added Q10, Q12, Q2, Q4, Q6, Q8: IRF520, transistor-power:TO220BV
- added R10, R12, R14, R4, R6, R8: 1k, rcl:0207/10
- added R11, R13, R3, R5, R7, R9: 10k, rcl:0207/10
- added SL4, SL5, SL6: (no value), con-amp-quick:09P
- added U$4: STEPDOWN3A, ReguladoresStep:REGULADORSTEP-DOWN3A
- added U$5: STEPDOWN3ADISPLAY, ReguladoresStep:REGULADORWITHDISPLAY
- added X10, X11, X7, X8, X9: (no value), con-ptr500:AK300/2
- added X12: (no value), con-ptr500:AK300/9
- added X2: KUSBVX, con-kycon:KUSBVX
- U$3: value STEPDOWN3A -> STEPDOWN5A; device ReguladoresStep:REGULADORSTEP-DOWN3/5A -> ReguladoresStep:REGULADORSTEP-DOWN5ACURRENT
- X3: value KUSBVX -> (none); device con-kycon:KUSBVX -> con-ptr500:AK300/2
- X5, X6: device con-ptr500:AK300/2 -> con-ptr500:AK300/9
- moved X6 302.9 mm to (-97.0, -8.00), turned to 270 degrees
- moved X5 242.6 mm to (-12.0, -61.5), flipped to the bottom
- moved X3 175.9 mm to (98.0, -55.8)
- moved U$3 131.4 mm to (90.8, 82.5), turned to 0 degrees
- moved C3 106.7 mm to (-2.56, 69.5), turned to 0 degrees
- moved X1 97.1 mm to (-2.56, 60.5), turned to 0 degrees
- moved C4 93.2 mm to (137.2, 8.31), turned to 180 degrees
- moved D1 88.7 mm to (147.9, -4.04), turned to 270 degrees
- moved X4 68.6 mm to (146.7, -55.3), turned to 90 degrees
- moved 3V3OUT 65.8 mm to (131.2, -50.4), turned to 270 degrees
- moved IC1 61.9 mm to (135.6, 6.60)
- moved 5VOUT 52.3 mm to (136.7, 15.1), turned to 180 degrees
- moved S1 51.6 mm to (141.2, -36.5)
- moved U$1 28.8 mm to (-27.8, 43.9)
- moved SV4 28.0 mm to (53.1, 40.7)
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Connections:
- new net 3V3MOT: MOTOR1.1, MOTOR1.3, MOTOR2.1, MOTOR2.3, MOTOR3.1, MOTOR3.3, MOTORIGHT.2, MOTORLEFT.2, U$4.P$3
- new net 5V5A: 5V5AOUT1.1, 5V5AOUT1.11, 5V5AOUT1.13, 5V5AOUT1.15, 5V5AOUT1.17, 5V5AOUT1.19, 5V5AOUT1.3, 5V5AOUT1.5, 5V5AOUT1.7, 5V5AOUT1.9, U$3.P$3
- new net ENDER: MOTORIGHT.5, MOTORIGHT.6, U$1.P34
- new net ENIZQ: MOTORLEFT.5, MOTORLEFT.6, U$1.P33
- new net GND@3: MOTOR1.2, MOTOR2.2, MOTOR3.2, MOTORIGHT.1, MOTORLEFT.1, U$4.P$4
- new net GND@4: 5V5AOUT1.10, 5V5AOUT1.12, 5V5AOUT1.14, 5V5AOUT1.16, 5V5AOUT1.18, 5V5AOUT1.2, 5V5AOUT1.20, 5V5AOUT1.4, 5V5AOUT1.6, 5V5AOUT1.8, U$3.P$4
- new net INA1: MOTOR1.6, U$1.P12
- new net INA2: MOTOR2.6, U$1.P32
- new net INA3: MOTOR3.6, U$1.P37
- new net INB1: MOTOR1.5, U$1.P11
- new net INB2: MOTOR2.5, U$1.P31
- new net INB3: MOTOR3.5, U$1.P36
- new net M1: D4.A, U$1.P2
- new net M2: D5.A, U$1.P3
- new net M3: D6.A, U$1.P4
- new net M4: D7.A, U$1.P8
- new net M5: D8.A, U$1.P9
- new net M6: D9.A, U$1.P10
- new net N$14: D1.A, F1.2A
- new net N$15: MOTOR2.4
- new net N$16: MOTOR3.4
- new net N$24: D4.C, Q1.B
- new net N$25: MOTOR1.4
- new net N$28: Q1.E, Q2.G, R3.1, R4.1
- new net N$30: LED1.A, R4.2
- new net N$31: D5.C, Q3.B
- new net N$39: Q2.D, X3.1
- new net N$40: SL4.9, U$1.P22, X5.1
- new net N$41: Q3.E, Q4.G, R5.1, R6.1
- new net N$42: LED2.A, R6.2
- new net N$43: Q4.D, X7.1
- new net N$44: D6.C, Q5.B
- new net N$45: Q5.E, Q6.G, R7.1, R8.1
- new net N$46: LED3.A, R8.2
- new net N$47: Q6.D, X8.1
- new net N$48: D7.C, Q7.B
- new net N$49: Q7.E, Q8.G, R10.1, R9.1
- new net N$50: LED4.A, R10.2
- new net N$51: Q8.D, X9.1
- new net N$52: D8.C, Q9.B
- new net N$53: Q10.G, Q9.E, R11.1, R12.1
- new net N$54: LED5.A, R12.2
- new net N$55: Q10.D, X10.1
- new net N$56: D9.C, Q11.B
- new net N$57: Q11.E, Q12.G, R13.1, R14.1
- new net N$58: LED6.A, R14.2
- new net N$59: Q12.D, X11.1
- new net N$60: SL4.8, U$1.P23, X5.2
- new net N$61: SL4.7, U$1.P24, X5.3
- new net N$62: SL4.6, U$1.P25, X5.4
- new net N$63: SL4.5, U$1.P26, X5.5
- new net N$64: SL4.4, U$1.P27, X5.6
- new net N$65: SL4.3, U$1.P28, X5.7
- new net N$66: SL4.2, U$1.P29, X5.8
- new net N$67: SL4.1, U$1.P30, X5.9
- new net N$68: SL6.9, U$1.P79, X12.1
- new net N$69: SL6.8, U$1.P78, X12.2
- new net N$70: SL6.7, U$1.P77, X12.3
- new net N$71: SL6.6, U$1.P76, X12.4
- new net N$72: SL6.5, U$1.P75, X12.5
- new net N$73: SL6.4, U$1.P74, X12.6
- new net N$74: SL6.3, U$1.P73, X12.7
- new net N$75: SL6.2, U$1.P72, X12.8
- new net N$76: SL6.1, U$1.P71, X12.9
- new net N$77: SL5.9, U$1.P59, X6.1
- new net N$78: SL5.8, U$1.P58, X6.2
- new net N$79: SL5.7, U$1.P57, X6.3
- new net N$80: SL5.6, U$1.P56, X6.4
- new net N$81: SL5.5, U$1.P55, X6.5
- new net N$82: SL5.4, U$1.P54, X6.6
- new net N$83: SL5.3, U$1.P53, X6.7
- new net N$84: SL5.2, U$1.P52, X6.8
- new net N$85: SL5.1, U$1.P51, X6.9
- new net N$86: ANALOGS.8, U$1.P63
- new net N$87: ANALOGS.7, U$1.P64
- new net N$88: ANALOGS.6, U$1.P65
- new net N$89: ANALOGS.5, U$1.P66
- new net N$90: ANALOGS.4, U$1.P67
- new net N$91: ANALOGS.3, U$1.P68
- new net N$92: ANALOGS.2, U$1.P69
- new net N$93: ANALOGS.1, U$1.P70
- new net PWM1: MOTORLEFT.8, U$1.P20
- new net PWM2: MOTORLEFT.7, U$1.P19
- new net PWM3: MOTORIGHT.8, U$1.P18
- new net PWM4: MOTORIGHT.7, U$1.P17
- new net PWM5: MOTOR2.7, U$1.P40
- new net PWM6: MOTOR3.7, U$1.P39
- new net PWM7: MOTOR1.7, U$1.P38
- net 5V1A: now also Q1.C, Q11.C, Q3.C, Q5.C, Q7.C, Q9.C
- net 5V3A: now also U$5.P$3, X2.1; no longer U$3.P$3
- net GND@1: now also C9.2, LED1.K, LED2.K, LED3.K, LED4.K, LED5.K, LED6.K, Q10.S, Q12.S, Q2.S, Q4.S, Q6.S, Q8.S, R11.2, R13.2, R3.2, R5.2, R7.2, R9.2, U$4.P$2, U$5.P$2
- net GND@2: now also U$5.P$4, X2.4; no longer U$3.P$4
- net N$2: now also F1.1A; no longer D1.A
- net N$5: now also C8.2
- net N$6: now also C8.1
- net VIN: now also C9.1, U$4.P$1, U$5.P$1, X10.2, X11.2, X3.2, X7.2, X8.2, X9.2
Routing:
- net 3V3MOT: track 0.00 -> 1079.3 mm
- net GND@1: track 0.00 -> 1061.4 mm, vias 0 -> 2
- net GND@3: track 0.00 -> 619.6 mm, vias 0 -> 2
- net VIN: track 0.00 -> 323.8 mm
- net PWM1: track 0.00 -> 301.8 mm
- net PWM2: track 0.00 -> 301.2 mm
- net PWM3: track 0.00 -> 295.6 mm
- net PWM4: track 0.00 -> 289.1 mm
- net 5V1A: track 0.00 -> 234.2 mm
- net M1: track 0.00 -> 154.6 mm
- net M2: track 0.00 -> 132.5 mm
- net M3: track 0.00 -> 113.2 mm
- net INB2: track 0.00 -> 111.7 mm, vias 0 -> 2
- net INA2: track 0.00 -> 109.6 mm, vias 0 -> 2
- net PWM7: track 0.00 -> 93.5 mm, vias 0 -> 2
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Other:
- board size 213.3 x 115.2 mm -> 273 x 160.3 mm

Commit message: BoardMiddle without optimization and review
Parts:
- moved X5 15.1 mm to (-10.5, -76.5)
- moved MOTORIGHT 15.0 mm to (-50.4, -70.3)
- moved MOTORLEFT 15.0 mm to (-50.4, -79.9)
- moved SL4 10.0 mm to (-11.6, -62.8)
Routing:
- net GND@3: track 619.6 -> 691.0 mm
- net 3V3MOT: track 1079.3 -> 1107.3 mm
- net PWM3: track 295.6 -> 318.1 mm
- net PWM1: track 301.8 -> 324.1 mm
- net PWM4: track 289.1 -> 311.2 mm
- net PWM2: track 301.2 -> 322.9 mm
- net N$40: track 66.7 -> 84.9 mm
- net N$60: track 61.3 -> 79.5 mm
- net N$61: track 56.7 -> 74.5 mm
- net N$62: track 51.9 -> 69.4 mm
- net N$63: track 47.4 -> 64.6 mm
- net N$64: track 44.5 -> 60.9 mm
- net N$65: track 41.8 -> 57.3 mm
- net N$66: track 39.1 -> 54.0 mm
- net ENDER: track 55.7 -> 69.7 mm
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Other:
- board size 273 x 160.3 mm -> 272 x 176.8 mm

Commit message: TIvaboardV1
Connections:
- removed net N$6: C1.+, C8.1, IC2.3
- removed net N$7: U$2.P14, U$2.P20, U$2.P25, U$2.P30, U$2.P34, U$2.P39, U$2.P6, U$2.P9
- net GND@1: now also SV4.15, U$2.P14, U$2.P20, U$2.P25, U$2.P30, U$2.P34, U$2.P39, U$2.P6, U$2.P9
- net VIN: now also C1.+, C8.1, IC2.3
Routing:
- net VIN: track 323.8 -> 405.8 mm
- net GND@1: track 1061.4 -> 1111.6 mm
- net N$6: track 28.6 -> 0.00 mm
- net M6: track 73.6 -> 58.9 mm
- net 5V5A: track 52.9 -> 62.0 mm
- net PWM1: track 324.1 -> 332.1 mm
- net M5: track 72.3 -> 66.1 mm
- net 5V1A: track 234.2 -> 240.1 mm
- net N$67: track 55.9 -> 60.6 mm
- net N$93: track 49.4 -> 54.0 mm
- net GND@3: track 691.0 -> 695.3 mm
- net 3V3MOT: track 1107.3 -> 1111.6 mm
- net N$92: track 45.6 -> 49.7 mm
- net PWM2: track 322.9 -> 326.4 mm
- net N$91: track 42.0 -> 45.5 mm
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- added copper zone on layer 16, net RASNET
Other:
- board text added: "SEEKER UCB TIVABOARD"
