File: Electronics/2024/TivaWareSeeker/CIRCUIT.sch (EAGLE design)
At the start: 29 parts, among them IC1 7805TV, X1 KUSBVX, X3 KUSBVX

Commit message: BoardMiddle
Parts:
- removed JP2, JP3, JP4: (no value), pinhead:PINHD-2X10
- removed SV1, SV2: (no value), con-lstb:MA10-1
- added 5V5AOUT1: (no value), pinhead:PINHD-2X10
- added ANALOGS: (no value), con-amp-quick:MA08
- added C8, C9: 0.1uF, rcl:C-EU075-052X106
- added D4, D5, D6, D7, D8, D9: 1N4004, diode:1N4004
- added F1: 6A, fuse:SHK20L
- added LED1, LED2, LED3, LED4, LED5, LED6: TLLG4400, led:TLLG4400
- added MOTOR1, MOTOR2, MOTOR3: (no value), con-amp-quick:MA07
- added MOTORIGHT, MOTORLEFT: (no value), pinhead:PINHD-2X4
- added Q1, Q11, Q3, Q5, Q7, Q9: BC548, transistor-npn:BC548
- added Q10, Q12, Q2, Q4, Q6, Q8: IRF520, transistor-power:IRF520
- added R10, R12, R14, R4, R6, R8: 1k, rcl:R-US_0207/10
- added R11, R13, R3, R5, R7, R9: 10k, rcl:R-US_0207/10
- added SL4, SL5, SL6: (no value), con-amp-quick:M09
- added U$4: STEPDOWN3A, ReguladoresStep:STEPDOWN3A
- added U$5: STEPDOWN3ADISPLAY, ReguladoresStep:STEPDOWN3ADISPLAY
- added X10, X11, X7, X8, X9: (no value), con-ptr500:AK300/2
- added X12: (no value), con-ptr500:AK300/9
- added X2: KUSBVX, con-kycon:KUSBVX
- U$3: value STEPDOWN3A -> STEPDOWN5A; device ReguladoresStep:STEPDOWN3A -> ReguladoresStep:STEPDOWN5A
- X3: value KUSBVX -> (none); device con-kycon:KUSBVX -> con-ptr500:AK300/2
- X5, X6: device con-ptr500:AK300/2 -> con-ptr500:AK300/9
Connections:
- new net 3V3MOT: MOTOR1.1, MOTOR1.3, MOTOR2.1, MOTOR2.3, MOTOR3.1, MOTOR3.3, MOTORIGHT.2, MOTORLEFT.2, U$4.VOUT+
- new net 5V5A: 5V5AOUT1.1, 5V5AOUT1.11, 5V5AOUT1.13, 5V5AOUT1.15, 5V5AOUT1.17, 5V5AOUT1.19, 5V5AOUT1.3, 5V5AOUT1.5, 5V5AOUT1.7, 5V5AOUT1.9, U$3.VOUT+
- new net ENDER: MOTORIGHT.5, MOTORIGHT.6, U$1.PH0
- new net ENIZQ: MOTORLEFT.5, MOTORLEFT.6, U$1.PH1
- new net GND@3: MOTOR1.2, MOTOR2.2, MOTOR3.2, MOTORIGHT.1, MOTORLEFT.1, U$4.VOUT-
- new net GND@4: 5V5AOUT1.10, 5V5AOUT1.12, 5V5AOUT1.14, 5V5AOUT1.16, 5V5AOUT1.18, 5V5AOUT1.2, 5V5AOUT1.20, 5V5AOUT1.4, 5V5AOUT1.6, 5V5AOUT1.8, U$3.VOUT-
- new net INA1: MOTOR1.6, U$1.PL2
- new net INA2: MOTOR2.6, U$1.PK6
- new net INA3: MOTOR3.6, U$1.PM0
- new net INB1: MOTOR1.5, U$1.PL3
- new net INB2: MOTOR2.5, U$1.PK7
- new net INB3: MOTOR3.5, U$1.PM1
- new net M1: D4.A, U$1.PM3
- new net M2: D5.A, U$1.PH2
- new net M3: D6.A, U$1.PH3
- new net M4: D7.A, U$1.PN2
- new net M5: D8.A, U$1.PN3
- new net M6: D9.A, U$1.PP2
- new net N$14: D1.A, F1.2A
- new net N$15: MOTOR2.4
- new net N$16: MOTOR3.4
- new net N$24: D4.C, Q1.B
- new net N$25: MOTOR1.4
- new net N$28: Q1.E, Q2.G, R3.1, R4.1
- new net N$30: LED1.A, R4.2
- new net N$31: D5.C, Q3.B
- new net N$39: Q2.D, X3-1.KL
- new net N$40: SL4.9, U$1.PM7, X5-1.KL
- new net N$41: Q3.E, Q4.G, R5.1, R6.1
- new net N$42: LED2.A, R6.2
- new net N$43: Q4.D, X7-1.KL
- new net N$44: D6.C, Q5.B
- new net N$45: Q5.E, Q6.G, R7.1, R8.1
- new net N$46: LED3.A, R8.2
- new net N$47: Q6.D, X8-1.KL
- new net N$48: D7.C, Q7.B
- new net N$49: Q7.E, Q8.G, R10.1, R9.1
- new net N$50: LED4.A, R10.2
- new net N$51: Q8.D, X9-1.KL
- new net N$52: D8.C, Q9.B
- new net N$53: Q10.G, Q9.E, R11.1, R12.1
- new net N$54: LED5.A, R12.2
- new net N$55: Q10.D, X10-1.KL
- new net N$56: D9.C, Q11.B
- new net N$57: Q11.E, Q12.G, R13.1, R14.1
- new net N$58: LED6.A, R14.2
- new net N$59: Q12.D, X11-1.KL
- new net N$60: SL4.8, U$1.PP5, X5-2.KL
- new net N$61: SL4.7, U$1.TX2/PA7, X5-3.KL
- new net N$62: SL4.6, U$1.RESET@2, X5-4.KL
- new net N$63: SL4.5, U$1.MOSI6/PQ2, X5-5.KL
- new net N$64: SL4.4, U$1.MISO6/PQ3, X5-6.KL
- new net N$65: SL4.3, U$1.PP3, X5-7.KL
- new net N$66: SL4.2, U$1.CS5/PQ1, X5-8.KL
- new net N$67: SL4.1, U$1.PM6, X5-9.KL
- new net N$68: SL6.9, U$1.MOSI1/A9/PE4, X12-1.KL
- new net N$69: SL6.8, U$1.RX7/PC4, X12-2.KL
- new net N$70: SL6.7, U$1.TX7/PC5, X12-3.KL
- new net N$71: SL6.6, U$1.RX5/PC6, X12-4.KL
- new net N$72: SL6.5, U$1.MISO1/A8/PE5, X12-5.KL
- new net N$73: SL6.4, U$1.CLK2/A12/PD3, X12-6.KL
- new net N$74: SL6.3, U$1.TX5/PC7, X12-7.KL
- new net N$75: SL6.2, U$1.SCL0/PB2, X12-8.KL
- new net N$76: SL6.1, U$1.SDA0/PB3, X12-9.KL
- new net N$77: SL5.9, U$1.CS/A13/PD2, X6-1.KL
- new net N$78: SL5.8, U$1.RX6/PP0, X6-2.KL
- new net N$79: SL5.7, U$1.TX6/PP1, X6-3.KL
- new net N$80: SL5.6, U$1.A7/PD4, X6-4.KL
- new net N$81: SL5.5, U$1.A6/PD5, X6-5.KL
- new net N$82: SL5.4, U$1.CLK5/PQ0, X6-6.KL
- new net N$83: SL5.3, U$1.PP4, X6-7.KL
- new net N$84: SL5.2, U$1.SCL1/PN5, X6-8.KL
- new net N$85: SL5.1, U$1.SDA1/PN4, X6-9.KL
- new net N$86: ANALOGS.8, U$1.A3/PE0
- new net N$87: ANALOGS.7, U$1.A2/PE1
- new net N$88: ANALOGS.6, U$1.A1/PE2
- new net N$89: ANALOGS.5, U$1.A0/PE3
- new net N$90: ANALOGS.4, U$1.A4/PD7
- new net N$91: ANALOGS.3, U$1.PA6
- new net N$92: ANALOGS.2, U$1.PM4
- new net N$93: ANALOGS.1, U$1.PM5
- new net PWM1: MOTORLEFT.8, U$1.PF1
- new net PWM2: MOTORLEFT.7, U$1.PF2
- new net PWM3: MOTORIGHT.8, U$1.PF3
- new net PWM4: MOTORIGHT.7, U$1.SCL1/PG0
- new net PWM5: MOTOR2.7, U$1.SDA1/PG1
- new net PWM6: MOTOR3.7, U$1.PK4
- new net PWM7: MOTOR1.7, U$1.PK5
- net 5V1A: now also Q1.C, Q11.C, Q3.C, Q5.C, Q7.C, Q9.C
- net 5V3A: now also U$5.VOUT+, X2.1; no longer U$3.VOUT+
- net GND@1: now also C9.2, LED1.C, LED2.C, LED3.C, LED4.C, LED5.C, LED6.C, Q10.S, Q12.S, Q2.S, Q4.S, Q6.S, Q8.S, R11.2, R13.2, R3.2, R5.2, R7.2, R9.2, U$4.VIN-, U$5.VIN-
- net GND@2: now also U$5.VOUT-, X2.4; no longer U$3.VOUT-
- net N$2: now also F1.1A; no longer D1.A
- net N$5: now also C8.2
- net N$6: now also C8.1
- net VIN: now also C9.1, U$4.VIN+, U$5.VIN+, X10-2.KL, X11-2.KL, X3-2.KL, X7-2.KL, X8-2.KL, X9-2.KL
Other:
- moved on the sheet: 3V3OUT, 5VOUT, C1, C2, C3, C4, D1, IC1, IC2, R1, R2, S1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

Commit message: TIvaboardV1
Connections:
- removed net N$6: C1.+, C8.1, IC2.IN
- removed net N$7: U$2.GND
- net GND@1: now also SV4.15, U$2.GND
- net VIN: now also C1.+, C8.1, IC2.IN
Changed lines of the file:
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@@
-</segment>
-<segment>
-<label x="-2.54" y="-195.58" size="1.778" layer="95" rot="MR0" xref="yes"/>
 </segment>
 <segment>
@@
 <pinref part="U$3" gate="G$1" pin="VIN+"/>
 </segment>
+<segment>
+<pinref part="C1" gate="G$1" pin="+"/>
+<pinref part="IC2" gate="A" pin="IN"/>
+<wire x1="22.86" y1="-200.66" x2="22.86" y2="-195.58" width="0.1524" layer="91"/>
+<wire x1="22.86" y1="-195.58" x2="30.48" y2="-195.58" width="0.1524" layer="91"/>
+<wire x1="2.54" y1="-195.58" x2="10.16" y2="-195.58" width="0.1524" layer="91"/>
+<junction x="22.86" y="-195.58"/>
+<pinref part="C8" gate="G$1" pin="1"/>
+<wire x1="10.16" y1="-195.58" x2="22.86" y2="-195.58" width="0.1524" layer="91"/>
+<wire x1="10.16" y1="-200.66" x2="10.16" y2="-195.58" width="0.1524" layer="91"/>
+<junction x="10.16" y="-195.58"/>
+<label x="2.54" y="-195.58" size="1.778" layer="95"/>
+</segment>
 </net>
 <net name="GND@1" class="7">
@@
 <segment>
 <label x="38.1" y="-226.06" size="1.778" layer="95" rot="MR270" xref="yes"/>
-</segment>
-<segment>
-<label x="152.4" y="22.86" size="1.778" layer="95" rot="MR180" xref="yes"/>
 </segment>
 <segment>
@@
 <pinref part="Q12" gate="G$1" pin="S"/>
 <wire x1="425.45" y1="-201.93" x2="425.45" y2="-224.79" width="0.1524" layer="91"/>
+</segment>
+<segment>
+<pinref part="U$2" gate="G$1" pin="GND"/>
+<wire x1="147.32" y1="22.86" x2="152.4" y2="22.86" width="0.1524" layer="91"/>
+<label x="152.4" y="22.86" size="1.778" layer="95"/>
+</segment>
+<segment>
+<pinref part="SV4" gate="1" pin="15"/>
+<wire x1="167.64" y1="-7.62" x2="165.1" y2="-7.62" width="0.1524" layer="91"/>
+<label x="157.48" y="-7.62" size="1.778" layer="95"/>
 </segment>
 </net>
@@
 </segment>
 </net>
-<net name="N$6" class="0">
-<segment>
-<pinref part="C1" gate="G$1" pin="+"/>
-<pinref part="IC2" gate="A" pin="IN"/>
-<wire x1="22.86" y1="-200.66" x2="22.86" y2="-195.58" width="0.1524" layer="91"/>
-<wire x1="22.86" y1="-195.58" x2="30.48" y2="-195.58" width="0.1524" layer="91"/>
-<wire x1="2.54" y1="-195.58" x2="10.16" y2="-195.58" width="0.1524" layer="91"/>
-<junction x="22.86" y="-195.58"/>
-<pinref part="C8" gate="G$1" pin="1"/>
-<wire x1="10.16" y1="-195.58" x2="22.86" y2="-195.58" width="0.1524" layer="91"/>
-<wire x1="10.16" y1="-200.66" x2="10.16" y2="-195.58" width="0.1524" layer="91"/>
-<junction x="10.16" y="-195.58"/>
-</segment>
-</net>
-<net name="N$7" class="0">
-<segment>
-<pinref part="U$2" gate="G$1" pin="GND"/>
-<wire x1="147.32" y1="22.86" x2="152.4" y2="22.86" width="0.1524" layer="91"/>
-</segment>
-</net>
